File: hardware/b4-carrier/b4-carrier.kicad_pcb (KiCad board)
At the start: 2 copper layers, 160 x 100 mm, 101 parts, among them J1 USB-C PD 12V, J10 ESP32 L, J11 ESP32 R 22.86, J12 ESP32 R 25.40, J13 ESP32 R 27.94, J2 DC 12V, J3 LENS 12-pin, J4 POT IRIS, J5 POT ZOOM, J6 POT FOCUS, J7 ZOOM DEMAND, J8 FOCUS DEMAND, J9 OLED cable, U1 CH224A, U2 L7809, U3 R-78E5.0-0.5, U4 LP2950CZ-3.3, U5 LM324, U6 ADS1115, U7 MCP4728 JP1, U8 MCP4728 JP2, U9 OLED

Commit message: Hardware B4-Traeger: ESP32-S3-ETH als Alternative, Fokus-Poti, Zoom 100k/180k, SPICE-Simulation
Simulation (ngspice): Iris-Stufe trifft die Bankmessung auf 0,1 V; alte
Zoomstufe verschiebt den Stopp um 227 mV je Volt der 9-V-Spannung, die neue
um 0; 100k/180k statt 10k/18k, damit die 5-V-Referenz des Objektivs nicht
belastet wird.

Co-Authored-By: Claude Opus 5.5 <noreply@anthropic.com>
Parts:
- added J14: S3-ETH IO20 row, PinSocket_1x20_P2.54mm_Vertical, F.Cu at (161.0, 28.0)
- added J15: S3-ETH VBUS row, PinSocket_1x20_P2.54mm_Vertical, F.Cu at (178.8, 28.0)
- added JP4: FOCUS POT, PinHeader_1x03_P2.54mm_Vertical, F.Cu at (135.0, 75.0)
- added RV3: 10k lin FOCUS, Potentiometer_Alps_RK09K_Single_Vertical, F.Cu at (132.8, 85.0)
- R20, R22, R30, R32: value 10k -> 100k
- R21, R23, R31, R33: value 18k -> 180k
- moved H2 24.0 mm to (180.0, 4.00)
- moved H4 24.0 mm to (180.0, 96.0)
Connections:
- R52 pad 1: EXT_F -> PF
Routing:
- net GND: track 809.4 -> 951.6 mm
- net SCL: track 122.3 -> 170.6 mm, vias 0 -> 1
- net A3V3: track 327.9 -> 368.8 mm
- net POT_I: track 44.8 -> 84.8 mm
- net SDA: track 132.0 -> 171.3 mm, vias 0 -> 1
- net POT_Z: track 51.0 -> 89.4 mm
- net ESP_VIN: track 137.6 -> 173.4 mm, vias 0 -> 1
- net EXT_F: track 66.6 -> 99.1 mm
- net PF: track 0.00 -> 31.6 mm
- net POT_F: track 46.0 -> 76.8 mm
- net DM: track 12.8 -> 26.4 mm, vias 2 -> 0
- net RV3W: track 0.00 -> 13.4 mm
- net V9: track 114.5 -> 125.9 mm, vias 2 -> 1
- net ZOOM_POS: track 106.4 -> 96.8 mm
- net IRIS_POS: track 95.3 -> 102.4 mm
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Other:
- board size 160 x 100 mm -> 184 x 100 mm
- board text added: "ESP32-S3-ETH"
- board text added: "ESP32-S3-ETH (+PoE) RJ45 ^"
- board text added: "ONLY ONE ESP32 BOARD"
